File: Hardware/KiCAD_Project_Files/BlueGiga_BLE112-IO_XBee_Module.sch (KiCad schematic (older format))
At the start: 14 parts, among them J1 CONNECTOR_USB_TYPE_MINI_B, P1 XBEE HEADER, P2 DEBUG, P3 HEADER_M_2.54MM_2R20P_ST_AU_P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, U1 BLE112-A, U2 AAT3221

Commit message: Rev 1.0 complete.  Updated all KiCAD project files and generated gerbers.
Parts:
- removed J1: CONNECTOR_USB_TYPE_MINI_B, Connector:CONNECTOR_USB_TYPE_MINI_B_RA_F_SMT_MOLEX, symbol CONNECTOR_USB_TYPE_MINI_B
- removed R1, R2: 33, Passive:0603, symbol RES_Small
- removed U2: AAT3221, Active:SOT23-5_SMT, symbol AAT3221
- P1: footprint Header:HEADER_50MIL_2R10P_SMT -> Header:HEADER_XBEE
Connections:
- net +3V3: no longer P2.9
- net USB+: no longer names the net of U1.11 (USB+)
- net USB-: no longer names the net of U1.12 (USB-)
- no-connect marks 19 -> 20
Other:
- note removed: "USB INTERFACE"
Changed lines of the file:
@@
 LIBS:TI_Luminary
 LIBS:TI_MSP430
-LIBS:BlueGiga_BLE112_XBee_GPIO_Module-cache
+LIBS:BlueGiga_BLE112-IO_XBee_Module-cache
 EELAYER 25 0
 EELAYER END
@@
 F 0 "P1" H 4575 6400 40  0000 C CNN
 F 1 "XBEE HEADER" H 4725 5150 40  0000 C CNN
-F 2 "Header:HEADER_50MIL_2R10P_SMT" H 5125 6200 60  0001 C CNN
+F 2 "Header:HEADER_XBEE" H 5125 6200 60  0001 C CNN
 F 3 "" H 5125 6200 60  0000 C CNN
 F 4 "S5800-40-ND" H 4725 5700 60  0001 C CNN "Digi-Key Part#"
@@
 $Comp
 L +3V3 #PWR010
-U 1 1 553BA15B
-P 9150 3625
-F 0 "#PWR010" H 9150 3475 50  0001 C CNN
-F 1 "+3V3" H 9150 3750 40  0000 C CNN
-F 2 "" H 9150 3625 60  0000 C CNN
-F 3 "" H 9150 3625 60  0000 C CNN
-	1    9150 3625
-	1    0    0    -1
-$EndComp
-$Comp
-L +3V3 #PWR011
 U 1 1 553BA2DC
 P 9950 3625
-F 0 "#PWR011" H 9950 3475 50  0001 C CNN
+F 0 "#PWR010" H 9950 3475 50  0001 C CNN
 F 1 "+3V3" H 9950 3750 40  0000 C CNN
 F 2 "" H 9950 3625 60  0000 C CNN
@@
 Text GLabel 3600 2700 0    40   Input ~ 0
 P1_6
-Text GLabel 3600 3000 0    40   Input ~ 0
-USB+
-Text GLabel 3600 3100 0    40   Input ~ 0
-USB-
 Text GLabel 3600 3200 0    40   Input ~ 0
 P1_5
@@
 Text GLabel 9825 5725 2    40   Input ~ 0
 P0_7
-Text GLabel 4950 7050 0    40   Input ~ 0
-USB+
-Text GLabel 4950 6950 0    40   Input ~ 0
-USB-
 Text GLabel 9275 5325 0    40   Input ~ 0
 P1_5
@@
 Text GLabel 5375 6050 2    40   Output ~ 0
 P0_5/RT
-$Comp
-L CONNECTOR_USB_TYPE_MINI_B J1
-U 1 1 559350D6
-P 5975 7050
-F 0 "J1" V 5965 7135 40  0000 C CNN
-F 1 "CONNECTOR_USB_TYPE_MINI_B" H 6000 6800 40  0001 C CNN
-F 2 "Connector:CONNECTOR_USB_TYPE_MINI_B_RA_F_SMT_MOLEX" H 5975 7050 60  0001 C CNN
-F 3 "" H 5975 7050 60  0000 C CNN
-F 4 "1 VBUS" V 5845 6935 20  0000 C CNN "Custom Field 1"
-F 5 "2 D-" V 5905 6915 20  0000 C CNN "Custom Field 2"
-F 6 "3 D+" V 5955 6915 20  0000 C CNN "Custom Field 3"
-F 7 "4 ID" V 6005 6905 20  0000 C CNN "Custom Field 4"
-F 8 "5 GND" V 6055 6925 20  0000 C CNN "Custom Field 5"
-	1    5975 7050
-	0    1    1    0
-$EndComp
-$Comp
-L AAT3221 U2
-U 1 1 559354C3
-P 4975 7450
-F 0 "U2" H 4775 7700 40  0000 C CNN
-F 1 "AAT3221" H 4775 7300 40  0000 C CNN
-F 2 "Active:SOT23-5_SMT" H 4975 7450 60  0001 C CNN
-F 3 "" H 4975 7450 60  0000 C CNN
-	1    4975 7450
-	-1   0    0    -1
-$EndComp
-$Comp
-L RES_Small R1
-U 1 1 55935609
-P 5450 6950
-F 0 "R1" H 5450 7000 40  0000 C CNN
-F 1 "33" H 5450 6900 40  0000 C CNN
-F 2 "Passive:0603" H 5450 6950 60  0001 C CNN
-F 3 "" H 5450 6950 60  0000 C CNN
-	1    5450 6950
-	1    0    0    -1
-$EndComp
-$Comp
-L RES_Small R2
-U 1 1 5593563B
-P 5325 7050
-F 0 "R2" H 5325 7100 40  0000 C CNN
-F 1 "33" H 5325 7000 40  0000 C CNN
-F 2 "Passive:0603" H 5325 7050 60  0001 C CNN
-F 3 "" H 5325 7050 60  0000 C CNN
-	1    5325 7050
-	1    0    0    -1
-$EndComp
-$Comp
-L GND #PWR012
-U 1 1 55935BA4
-P 4975 7700
-F 0 "#PWR012" H 4975 7700 30  0001 C CNN
-F 1 "GND" H 4975 7630 30  0001 C CNN
-F 2 "" H 4975 7700 60  0000 C CNN
-F 3 "" H 4975 7700 60  0000 C CNN
-	1    4975 7700
-	1    0    0    -1
-$EndComp
-$Comp
-L GND #PWR013
-U 1 1 559361AB
-P 5750 7700
-F 0 "#PWR013" H 5750 7700 30  0001 C CNN
-F 1 "GND" H 5750 7630 30  0001 C CNN
-F 2 "" H 5750 7700 60  0000 C CNN
-F 3 "" H 5750 7700 60  0000 C CNN
-	1    5750 7700
-	1    0    0    -1
-$EndComp
-$Comp
-L +3V3 #PWR014
-U 1 1 55936277
-P 4500 7250
-F 0 "#PWR014" H 4500 7100 50  0001 C CNN
-F 1 "+3V3" H 4500 7375 40  0000 C CNN
-F 2 "" H 4500 7250 60  0000 C CNN
-F 3 "" H 4500 7250 60  0000 C CNN
-	1    4500 7250
-	1    0    0    -1
-$EndComp
 Connection ~ 3325 5250
 Wire Wire Line
@@
 	9250 3725 9450 3725
 Wire Wire Line
-	9450 4125 9150 4125
-Wire Wire Line
-	9150 4125 9150 3625
-Wire Wire Line
 	9450 3825 9050 3825
 Wire Wire Line
@@
 	4000 2700 3600 2700
 Wire Wire Line
-	3600 3000 4000 3000
-Wire Wire Line
-	4000 3100 3600 3100
-Wire Wire Line
 	3600 3200 4000 3200
 Wire Wire Line
@@
 Wire Wire Line
 	9825 5725 9750 5725
-Wire Wire Line
-	5775 6950 5700 6950
-Wire Wire Line
-	5700 6950 5700 7300
-Wire Wire Line
-	5700 7300 5325 7300
-Wire Wire Line
-	5775 7000 5625 7000
-Wire Wire Line
-	5625 7000 5625 6950
-Wire Wire Line
-	5625 6950 5550 6950
-Wire Wire Line
-	5425 7050 5775 7050
-Wire Wire Line
-	5225 7050 4950 7050
-Wire Wire Line
-	4950 6950 5350 6950
-Wire Wire Line
-	5775 7150 5750 7150
-Wire Wire Line
-	5750 7150 5750 7700
-Wire Wire Line
-	4975 7700 4975 7650
-Wire Wire Line
-	4625 7300 4500 7300
-Wire Wire Line
-	4500 7300 4500 7250
-Wire Wire Line
-	5325 7450 5425 7450
-Wire Wire Line
-	5425 7450 5425 7300
-Connection ~ 5425 7300
-NoConn ~ 5775 7100
-NoConn ~ 4625 7450
 Text Notes 8650 4575 0    60   ~ 0
 2x8 - 100MIL BLE112 GPIO
 Wire Notes Line
-	8650 4625 8650 6200
-Wire Notes Line
-	8650 6200 10400 6200
-Wire Notes Line
-	10400 6200 10400 4625
+	8650 4625 8650 6075
+Wire Notes Line
+	8650 6075 10400 6075
+Wire Notes Line
+	10400 6075 10400 4625
 Wire Notes Line
 	10400 4625 8650 4625
-Text Notes 4350 6750 0    60   ~ 0
-USB INTERFACE
-Wire Notes Line
-	4350 6800 4350 7900
-Wire Notes Line
-	4350 7900 6150 7900
-Wire Notes Line
-	6150 7900 6150 6800
-Wire Notes Line
-	6150 6800 4350 6800
 Text GLabel 9275 5025 0    40   Input ~ 0
 P2_0
@@
 	9750 5825 10250 5825
 $Comp
-L +3V3 #PWR015
+L +3V3 #PWR011
 U 1 1 5599FD1D
 P 8825 4825
-F 0 "#PWR015" H 8825 4675 50  0001 C CNN
+F 0 "#PWR011" H 8825 4675 50  0001 C CNN
 F 1 "+3V3" H 8825 4950 40  0000 C CNN
 F 2 "" H 8825 4825 60  0000 C CNN
@@
 $EndComp
 $Comp
-L GND #PWR016
+L GND #PWR012
 U 1 1 5599FD44
 P 10250 5875
-F 0 "#PWR016" H 10250 5875 30  0001 C CNN
+F 0 "#PWR012" H 10250 5875 30  0001 C CNN
 F 1 "GND" H 10250 5805 30  0001 C CNN
 F 2 "" H 10250 5875 60  0000 C CNN
@@
 P 9550 5375
 F 0 "P3" H 9550 5925 40  0000 C CNN
-F 1 "HEADER_M_2.54MM_2R20P_ST_AU_PTH" H 9550 4825 40  0000 C CNN
+F 1 "HEADER_M_2.54MM_2R20P_ST_AU_PTH" H 9550 4825 40  0001 C CNN
 F 2 "Header:HEADER_100MIL_2R20P_EDGE" H 9550 5775 60  0001 C CNN
 F 3 "" H 9550 5775 60  0000 C CNN
@@
 $EndComp
 $Comp
-L GND #PWR017
+L GND #PWR013
 U 1 1 559F0A33
 P 3325 5800
-F 0 "#PWR017" H 3325 5800 30  0001 C CNN
+F 0 "#PWR013" H 3325 5800 30  0001 C CNN
 F 1 "GND" H 3325 5730 30  0001 C CNN
 F 2 "" H 3325 5800 60  0000 C CNN
@@
 	3325 5700 3325 5800
 $Comp
-L GND #PWR018
+L GND #PWR014
 U 1 1 559F0B4A
 P 3075 5800
-F 0 "#PWR018" H 3075 5800 30  0001 C CNN
+F 0 "#PWR014" H 3075 5800 30  0001 C CNN
 F 1 "GND" H 3075 5730 30  0001 C CNN
 F 2 "" H 3075 5800 60  0000 C CNN
@@
 	3075 5700 3075 5800
 $Comp
-L GND #PWR019
+L GND #PWR015
 U 1 1 559F14B9
 P 5500 3750
-F 0 "#PWR019" H 5500 3750 30  0001 C CNN
+F 0 "#PWR015" H 5500 3750 30  0001 C CNN
 F 1 "GND" H 5500 3680 30  0001 C CNN
 F 2 "" H 5500 3750 60  0000 C CNN
@@
 	5500 2400 5500 3750
 $Comp
-L GND #PWR020
+L GND #PWR016
 U 1 1 559F1BAA
 P 3900 3450
-F 0 "#PWR020" H 3900 3450 30  0001 C CNN
+F 0 "#PWR016" H 3900 3450 30  0001 C CNN
 F 1 "GND" H 3900 3380 30  0001 C CNN
 F 2 "" H 3900 3450 60  0000 C CNN
@@
 Wire Wire Line
 	3900 2000 3900 3450
+NoConn ~ 9450 4125
+NoConn ~ 4000 3000
+NoConn ~ 4000 3100
 $EndSCHEMATC

Commit message: Changed schematic and board layout to conform to BlueGiga's usage of USART1 ALT1.
Connections:
- net +3V3: now also P2.9
- net P0_2/RX: now also P3.14, U1.23 (P0_5); no longer P3.8, U1.26 (P0_2)
- net P0_3/TX: now also P3.12, U1.24 (P0_4); no longer P3.10, U1.25 (P0_3)
- net P0_4/CT: now also P3.8, U1.26 (P0_2); no longer P3.12, U1.24 (P0_4)
- net P0_5/RT: now also P3.10, U1.25 (P0_3); no longer P3.14, U1.23 (P0_5)
- no-connect marks 20 -> 19
Other:
- note added: "* Default configuration"
- note added: "USART1*"
- moved on the sheet: P2, P3
